File: i2c_frontpanel.sch (KiCad schematic (older format))
At the start: 28 parts

Commit message: Schematic done.
Parts:
- removed Q? (x4): Q_PMOS_GSD, symbol Q_PMOS_GSD
- added C? (x8): 0.1uF, symbol C
- added Q? (x4): 2N7002, TO_SOT_Packages_SMD:SOT-23, symbol 2N7002
- added R? (x13): 10k, symbol R
- added R? (x2): 4.7k, symbol R
- added R? (x34): 470, symbol R
- added R? (x6): 100, symbol R
Connections:
- net labels added: A, B, B1, B2, B3, B4, B5, B6, C, D, DP0, DP1, DP2, DP3, GND, LD0, LD1, LD2, LD3, LED1, LED2, MISO, MOSI, RST, S1, S2, S3, S4, S5, S6, SCK, SCL, SDA, SW1, SW2, SW3, SW4, SW5, SW6, VCC, Vcc
- wire segments 0 -> 332
- no-connect marks 0 -> 5
Other:
- moved on the sheet: CON?, IC?, U?

Commit message: Footprints done. LICENSE now CERN open hardware license.
Parts:
- removed AFF?: 7SEGMENTS, symbol 7SEGMENTS
- AFF1, AFF2, AFF3, AFF4: renamed from AFF?; footprint (none) -> i2c_frontpanel:7seg_LTS_4817CKR_P
- C1, C2, C3, C4, C5, C6, C7, C8: renamed from C?; footprint (none) -> Capacitors_SMD:C_1206
- CON1: renamed from CON?; footprint AVR-ISP-6 -> Pin_Headers:Pin_Header_Straight_SMT_02x03
- D1, D2: renamed from D?; footprint (none) -> LEDs:LED_1206
- IC1: renamed from IC?; footprint TQFP32 -> Housings_QFP:TQFP-32_7x7mm_Pitch0.8mm
- R1, R10, R11, R12, R13, R14, R15, R16, R17, R18, R19, R2, R20, R21, R22, R23, R24, R25, R26, R27, R28, R29, R3, R30, R31, R32, R33, R34, R35, R36, R37, R38, R39, R4, R40, R41, R42, R43, R44, R45, R46, R47, R48, R49, R5, R50, R51, R52, R53, R54, R55, R6, R7, R8, R9: renamed from R?; footprint (none) -> Resistors_SMD:R_1206
- U1: renamed from U?; footprint (none) -> SMD_Packages:SOIC-14_N
- U10, U11, U12, U13: renamed from U?; footprint (none) -> SMD_Packages:SO-16-N
- U2, U3, U4, U5, U6, U7: renamed from U?; footprint (none) -> Resistors_SMD:R_2816
- U8, U9: renamed from U?; footprint (none) -> Pin_Headers:Pin_Header_Straight_1x04
- gave numbers to parts that had none: 6
