File: 2x7seg_4btn.kicad_pcb (KiCad board)
At the start: 2 copper layers, 64 x 26.3 mm, 61 parts, among them CON1 AVR-ISP, IC1 ATTINY88-A, Q1 2N7002, Q2 2N7002, Q3 2N7002, Q4 2N7002, U1 74HC14D_653, U10 MC14543B, U11 MC14543B, U2 SW_SPST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

Commit message: v1.1 fixed 74HC14 bottom-row button pin mappings.
Parts:
- CON1: value AVR-ISP -> AVR-ISP-6-DR
- U8: value SCL SCA GND Vcc -> SCL SDA GND VCC
- U9: value SCL SDA GND Vcc -> SCL SDA GND VCC
Connections:
- U1 pad 10: /B5 -> /SW5
- U1 pad 11: /SW5 -> /B5
- U1 pad 12: /B6 -> /SW6
- U1 pad 13: /SW6 -> /B6
- U1 pad 8: /B4 -> /SW4
- U1 pad 9: /SW4 -> /B4
Routing:
- net /SW5: track 49.1 -> 50.5 mm
- net /SW6: track 48.1 -> 49.4 mm
- net /SW4: track 49.7 -> 51.0 mm
- net /B5: track 6.53 -> 7.71 mm
- net /B6: track 6.25 -> 5.72 mm
- net /B4: track 0.00 -> 0.51 mm
Other:
- board text added: "i2c frontpanel 2x7seg_4btn v1.1 - DVR"
- board text removed: "i2c frontpanel 2x7seg_4btn v1.0 - DVR"
