File: 4x7seg_6btn.kicad_pcb (KiCad board)
At the start: 2 copper layers, 91.8 x 26.3 mm, 94 parts, among them CON1 AVR-ISP, IC1 ATTINY88-A, Q1 2N7002, Q2 2N7002, Q3 2N7002, Q4 2N7002, Q5 2N7002, Q6 2N7002, U1 74HC14D_653, U10 MC14543B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

Commit message: v1.1 fixed 74HC14 bottom-row button pin mappings.
Parts:
- CON1: value AVR-ISP -> AVR-ISP-6-DR
- U8: value SCL SCA GND Vcc -> SCL SDA GND VCC
- U9: value SCL SDA GND Vcc -> SCL SDA GND VCC
Connections:
- U1 pad 10: /B5 -> /SW5
- U1 pad 11: /SW5 -> /B5
- U1 pad 12: /B6 -> /SW6
- U1 pad 13: /SW6 -> /B6
- U1 pad 8: /B4 -> /SW4
- U1 pad 9: /SW4 -> /B4
Routing:
- net /B4: track 10.4 -> 12.3 mm
- net /SW4: track 70.0 -> 71.4 mm
- net /SW6: track 68.4 -> 69.7 mm
- net /SW5: track 69.4 -> 70.7 mm
- net /B5: track 6.53 -> 7.71 mm
- net /B6: track 6.25 -> 5.72 mm
Other:
- board text added: "i2c frontpanel 4x7seg_6btn v1.1 - DVR"
- board text removed: "i2c frontpanel 4x7seg_6btn v1.0 - DVR"
